Commit message: Fixed URDF to use <LEG>_<SERVO> naming convention for important joints, adjusted visualize.py

File: rl_training/urdf/robot_dog.urdf (robot description, URDF)
Before this commit: robot robot_dog, 56 links, 55 joints
Joints:
- removed joint back-left-femur-femur/back-left-shin-shin
- removed joint back-left-femur-servo/disc
- removed joint back-left-femur-servo/front-left-hip
- removed joint back-left-pelvis-servo/disc
- removed joint back-right-femur-femur/back-right-shin-shin
- removed joint back-right-femur-servo/disc
- removed joint back-right-pelvis-servo/disc
- removed joint front-left-femur-femur/front-left-shin-shin
- removed joint front-left-femur-servo/disc
- removed joint front-left-pelvis-servo/disc
- removed joint front-right-femur-femur/front-right-shin-shin
- removed joint front-right-femur-servo/disc
- removed joint front-right-pelvis-servo/disc
- added joint BL_hip: type revolute, parent back-left-pelvis-servo, child back-left-pelvis-disc, origin xyz=0 -0.00995 0.04605 rpy=0 0 -0.349066, axis 0 0 1, limit lower=-0.349066 upper=0.349066 effort=5.0 velocity=9.52
- added joint BL_lower: type continuous, parent back-left-femur-femur, child back-left-shin-shin, origin xyz=0.0076 0.07777 -0.07777 rpy=0 0 0
- added joint BL_upper: type continuous, parent back-left-femur-servo, child back-left-femur-disc, origin xyz=0 -0.01 0.047 rpy=0 0 0, axis 0 0 1
- added joint BR_hip: type revolute, parent back-right-pelvis-servo, child back-right-pelvis-disc, origin xyz=0 -0.0106 0.04605 rpy=0 0 0.349066, axis 0 0 1, limit lower=-0.349066 upper=0.349066 effort=5.0 velocity=9.52
- added joint BR_lower: type continuous, parent back-right-femur-femur, child back-right-shin-shin, origin xyz=-0.0076 0.07777 -0.07777 rpy=0 0 0
- added joint BR_upper: type continuous, parent back-right-femur-servo, child back-right-femur-disc, origin xyz=0 -0.01 0.047 rpy=0 0 0, axis 0 0 1
- added joint FL_hip: type revolute, parent front-left-pelvis-servo, child front-left-pelvis-disc, origin xyz=0 -0.00995 0.04605 rpy=0 0 0.349066, axis 0 0 1, limit lower=-0.349066 upper=0.349066 effort=5.0 velocity=9.52
- added joint FL_lower: type continuous, parent front-left-femur-femur, child front-left-shin-shin, origin xyz=0.0076 0.07777 -0.07777 rpy=0 0 0
- added joint FL_upper: type continuous, parent front-left-femur-servo, child front-left-femur-disc, origin xyz=0 -0.01 0.047 rpy=0 0 0, axis 0 0 1
- added joint FR_hip: type revolute, parent front-right-pelvis-servo, child front-right-pelvis-disc, origin xyz=0 -0.0106 0.04605 rpy=0 0 -0.349066, axis 0 0 1, limit lower=-0.349066 upper=0.349066 effort=5.0 velocity=9.52
- added joint FR_lower: type continuous, parent front-right-femur-femur, child front-right-shin-shin, origin xyz=-0.0076 0.07777 -0.07777 rpy=0 0 0
- added joint FR_upper: type continuous, parent front-right-femur-servo, child front-right-femur-disc, origin xyz=0 -0.01 0.047 rpy=0 0 0, axis 0 0 1
- added joint back-left-femur-servo/back-left-hip: type continuous, parent back-left-femur-servo, child back-left-hip, origin xyz=0 -0.01 0.0409 rpy=0 -1.5708 3.14

Commit message: Made accurate ranges for all relevant joints

File: rl_training/urdf/robot_dog.urdf (robot description, URDF)
Before this commit: robot robot_dog, 56 links, 55 joints
Joints:
- joint BL_hip: origin xyz=0 -0.00995 0.04605 rpy=0 0 -0.349066 -> xyz=0 -0.00995 0.04605 rpy=0 0 0
- joint BL_lower: axis (none) -> 1 0 0; limit (none) -> lower=-0.698 upper=0.698 effort=5.0 velocity=9.52; type continuous -> revolute
- joint BL_upper: limit (none) -> lower=-0.654 upper=0.654 effort=5.0 velocity=9.52; type continuous -> revolute
- joint BR_hip: origin xyz=0 -0.0106 0.04605 rpy=0 0 0.349066 -> xyz=0 -0.0106 0.04605 rpy=0 0 0
- joint BR_lower: axis (none) -> 1 0 0; limit (none) -> lower=-0.698 upper=0.698 effort=5.0 velocity=9.52
- joint BR_upper: limit (none) -> lower=-0.654 upper=0.654 effort=5.0 velocity=9.52
- joint FL_hip: origin xyz=0 -0.00995 0.04605 rpy=0 0 0.349066 -> xyz=0 -0.00995 0.04605 rpy=0 0 0
- joint FL_lower: axis (none) -> 1 0 0; limit (none) -> lower=-0.698 upper=0.698 effort=5.0 velocity=9.52; type continuous -> revolute
- joint FL_upper: limit (none) -> lower=-0.654 upper=0.654 effort=5.0 velocity=9.52; type continuous -> revolute
- joint FR_hip: origin xyz=0 -0.0106 0.04605 rpy=0 0 -0.349066 -> xyz=0 -0.0106 0.04605 rpy=0 0 0
- joint FR_lower: axis (none) -> 1 0 0; limit (none) -> lower=-0.698 upper=0.698 effort=5.0 velocity=9.52; type continuous -> revolute
- joint FR_upper: limit (none) -> lower=-0.654 upper=0.654 effort=5.0 velocity=9.52; type continuous -> revolute

Commit message: Finished URDF

File: rl_training/urdf/robot_dog.urdf (robot description, URDF)
Before this commit: robot robot_dog, 56 links, 55 joints
Joints:
- joint BR_lower: axis 1 0 0 -> -1 0 0; type continuous -> revolute
- joint BR_upper: type continuous -> revolute
- joint FR_lower: axis 1 0 0 -> -1 0 0
