Commit message: Going to sack the thread based movement because isaac sim is doesnt like it, saving before cursor

File: training/urdf/robot_dog_OLD.urdf (robot description, URDF)
Before this commit: robot Robot_Dog, 48 links, 47 joints
Links:
- added link back_left_hip, mass 0.01; collision mesh filename=/home/matthewthomasbeck/Projects/Robot_Dog/training/meshes/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 scale=1 1 1; visual mesh filename=/home/matthewthomasbeck/Projects/Robot_Dog/training/meshes/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 scale=1 1 1
- added link back_left_shin_horn, mass 0.01; collision mesh filename=/home/matthewthomasbeck/Projects/Robot_Dog/training/meshes/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 scale=1 1 1; visual mesh filename=/home/matthewthomasbeck/Projects/Robot_Dog/training/meshes/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 scale=1 1 1
- added link back_right_hip, mass 0.01; collision mesh filename=/home/matthewthomasbeck/Projects/Robot_Dog/training/meshes/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 scale=1 1 1; visual mesh filename=/home/matthewthomasbeck/Projects/Robot_Dog/training/meshes/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 scale=1 1 1
- added link back_right_shin_horn, mass 0.01; collision mesh filename=/home/matthewthomasbeck/Projects/Robot_Dog/training/meshes/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 scale=1 1 1; visual mesh filename=/home/matthewthomasbeck/Projects/Robot_Dog/training/meshes/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 scale=1 1 1
- added link front_left_hip, mass 0.01; collision mesh filename=/home/matthewthomasbeck/Projects/Robot_Dog/training/meshes/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 scale=1 1 1; visual mesh filename=/home/matthewthomasbeck/Projects/Robot_Dog/training/meshes/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 scale=1 1 1
- added link front_left_shin_horn, mass 0.01; collision mesh filename=/home/matthewthomasbeck/Projects/Robot_Dog/training/meshes/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 scale=1 1 1; visual mesh filename=/home/matthewthomasbeck/Projects/Robot_Dog/training/meshes/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 scale=1 1 1
- added link front_right_hip, mass 0.01; collision mesh filename=/home/matthewthomasbeck/Projects/Robot_Dog/training/meshes/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 scale=1 1 1; visual mesh filename=/home/matthewthomasbeck/Projects/Robot_Dog/training/meshes/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 scale=1 1 1
- added link front_right_shin_horn, mass 0.01; collision mesh filename=/home/matthewthomasbeck/Projects/Robot_Dog/training/meshes/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 scale=1 1 1; visual mesh filename=/home/matthewthomasbeck/Projects/Robot_Dog/training/meshes/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 scale=1 1 1
Joints:
- added joint back_left_femur_servo_back_left_hip: type continuous, parent back_left_femur_servo, child back_left_hip, origin xyz=0 -0.01 0.0409 rpy=0 -1.5708 3.14
- added joint back_left_shin_servo_horn: type continuous, parent back_left_shin_servo, child back_left_shin_horn, origin xyz=0 -0.01 0.043 rpy=0 0 0.785398, axis 0 0 1
- added joint back_right_femur_servo_back_right_hip: type continuous, parent back_right_femur_servo, child back_right_hip, origin xyz=0 -0.01 0.0468 rpy=0 1.5708 3.14
- added joint back_right_shin_servo_horn: type continuous, parent back_right_shin_servo, child back_right_shin_horn, origin xyz=0 -0.01 0.043 rpy=0 0 2.356198, axis 0 0 1
- added joint front_left_femur_servo_front_left_hip: type continuous, parent front_left_femur_servo, child front_left_hip, origin xyz=0 -0.01 0.0409 rpy=0 -1.5708 3.14
- added joint front_left_shin_servo_horn: type continuous, parent front_left_shin_servo, child front_left_shin_horn, origin xyz=0 -0.01 0.043 rpy=0 0 0.785398, axis 0 0 1
- added joint front_right_femur_servo_front_right_hip: type continuous, parent front_right_femur_servo, child front_right_hip, origin xyz=0 -0.01 0.0468 rpy=0 1.5708 3.14
- added joint front_right_shin_servo_horn: type continuous, parent front_right_shin_servo, child front_right_shin_horn, origin xyz=0 -0.01 0.043 rpy=0 0 2.356198, axis 0 0 1
