Commit message: Cleaned up training space, I have to do it here because of context

File: training/urdf/robot_dog.urdf (robot description, URDF)
Before this commit: robot robot_dog, 56 links, 55 joints
Links:
- link midsection-bottom: geometry collision mesh filename=meshes/midsection/ares_midsection-bottom_1.0.dae scale=1 1 1; visual mesh filename=meshes/midsection/ares_midsection-bottom_1.0.dae scale=1 1 1
