Commit message: Got URDF loaded and working with Isaac Sim!

File: training/urdf/robot_dog.urdf (robot description, URDF)
Before this commit: robot robot_dog, 56 links, 55 joints
Links:
- removed link ai_module-mock
- removed link back-butt
- removed link back-left-femur-disc
- removed link back-left-femur-femur
- removed link back-left-femur-servo
- removed link back-left-foot
- removed link back-left-hip
- removed link back-left-pelvis-disc
- removed link back-left-pelvis-pelvis
- removed link back-left-pelvis-servo
- removed link back-left-shin-horn
- removed link back-left-shin-servo
- removed link back-left-shin-shin
- removed link back-right-femur-disc
- removed link back-right-femur-femur
- removed link back-right-femur-servo
- removed link back-right-foot
- removed link back-right-hip
- removed link back-right-pelvis-disc
- removed link back-right-pelvis-pelvis
- removed link back-right-pelvis-servo
- removed link back-right-shin-horn
- removed link back-right-shin-servo
- removed link back-right-shin-shin
- removed link back-top
- removed link front-face
- removed link front-left-femur-disc
- removed link front-left-femur-femur
- removed link front-left-femur-servo
- removed link front-left-foot
- removed link front-left-hip
- removed link front-left-pelvis-disc
- removed link front-left-pelvis-pelvis
- removed link front-left-pelvis-servo
- removed link front-left-shin-horn
- removed link front-left-shin-servo
- removed link front-left-shin-shin
- removed link front-right-femur-disc
- removed link front-right-femur-femur
- removed link front-right-femur-servo
- removed link front-right-foot
- removed link front-right-hip
- removed link front-right-pelvis-disc
- removed link front-right-pelvis-pelvis
- removed link front-right-pelvis-servo
- removed link front-right-shin-horn
- removed link front-right-shin-servo
- removed link front-right-shin-shin
- removed link front-top
- removed link midsection-batteryplate
- removed link midsection-bottom
- removed link midsection-connectorplate
- removed link midsection-side-left
- removed link midsection-side-right
- removed link midsection-top
- added link ai_module_mock, mass 0.01; collision mesh filename=/home/matthewthomasbeck/Projects/Robot_Dog/training/meshes/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 scale=1 1 1; visual mesh filename=/home/matthewthomasbeck/Projects/Robot_Dog/training/meshes/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 scale=1 1 1
- added link back_butt, mass 0.01; collision mesh filename=/home/matthewthomasbeck/Projects/Robot_Dog/training/meshes/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 scale=1 1 1; visual mesh filename=/home/matthewthomasbeck/Projects/Robot_Dog/training/meshes/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 scale=1 1 1
- added link back_left_femur_disc, mass 0.01; collision mesh filename=/home/matthewthomasbeck/Projects/Robot_Dog/training/meshes/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 scale=1 1 1; visual mesh filename=/home/matthewthomasbeck/Projects/Robot_Dog/training/meshes/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 scale=1 1 1
- added link back_left_femur_femur, mass 0.01; collision mesh filename=/home/matthewthomasbeck/Projects/Robot_Dog/training/meshes/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 scale=1 1 1; visual mesh filename=/home/matthewthomasbeck/Projects/Robot_Dog/training/meshes/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 scale=1 1 1
- added link back_left_femur_servo, mass 0.01; collision mesh filename=/home/matthewthomasbeck/Projects/Robot_Dog/training/meshes/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 scale=1 1 1; visual mesh filename=/home/matthewthomasbeck/Projects/Robot_Dog/training/meshes/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 scale=1 1 1
- added link back_left_foot, mass 0.01; collision mesh filename=/home/matthewthomasbeck/Projects/Robot_Dog/training/meshes/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 scale=1 1 1; visual mesh filename=/home/matthewthomasbeck/Projects/Robot_Dog/training/meshes/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 scale=1 1 1
- added link back_left_hip, mass 0.01; collision mesh filename=/home/matthewthomasbeck/Projects/Robot_Dog/training/meshes/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 scale=1 1 1; visual mesh filename=/home/matthewthomasbeck/Projects/Robot_Dog/training/meshes/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 scale=1 1 1
- added link back_left_pelvis_disc, mass 0.01; collision mesh filename=/home/matthewthomasbeck/Projects/Robot_Dog/training/meshes/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 scale=1 1 1; visual mesh filename=/home/matthewthomasbeck/Projects/Robot_Dog/training/meshes/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 scale=1 1 1
- added link back_left_pelvis_pelvis, mass 0.01; collision mesh filename=/home/matthewthomasbeck/Projects/Robot_Dog/training/meshes/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 scale=1 1 1; visual mesh filename=/home/matthewthomasbeck/Projects/Robot_Dog/training/meshes/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 scale=1 1 1
- added link back_left_pelvis_servo, mass 0.01; collision mesh filename=/home/matthewthomasbeck/Projects/Robot_Dog/training/meshes/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 scale=1 1 1; visual mesh filename=/home/matthewthomasbeck/Projects/Robot_Dog/training/meshes/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 scale=1 1 1
- added link back_left_shin_horn, mass 0.01; collision mesh filename=/home/matthewthomasbeck/Projects/Robot_Dog/training/meshes/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 scale=1 1 1; visual mesh filename=/home/matthewthomasbeck/Projects/Robot_Dog/training/meshes/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 scale=1 1 1
- added link back_left_shin_servo, mass 0.01; collision mesh filename=/home/matthewthomasbeck/Projects/Robot_Dog/training/meshes/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 scale=1 1 1; visual mesh filename=/home/matthewthomasbeck/Projects/Robot_Dog/training/meshes/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 scale=1 1 1
- added link back_left_shin_shin, mass 0.01; collision mesh filename=/home/matthewthomasbeck/Projects/Robot_Dog/training/meshes/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 scale=1 1 1; visual mesh filename=/home/matthewthomasbeck/Projects/Robot_Dog/training/meshes/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 scale=1 1 1
- added link back_right_femur_disc, mass 0.01; collision mesh filename=/home/matthewthomasbeck/Projects/Robot_Dog/training/meshes/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 scale=1 1 1; visual mesh filename=/home/matthewthomasbeck/Projects/Robot_Dog/training/meshes/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 scale=1 1 1
- added link back_right_femur_femur, mass 0.01; collision mesh filename=/home/matthewthomasbeck/Projects/Robot_Dog/training/meshes/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 scale=1 1 1; visual mesh filename=/home/matthewthomasbeck/Projects/Robot_Dog/training/meshes/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 scale=1 1 1
- added link back_right_femur_servo, mass 0.01; collision mesh filename=/home/matthewthomasbeck/Projects/Robot_Dog/training/meshes/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 scale=1 1 1; visual mesh filename=/home/matthewthomasbeck/Projects/Robot_Dog/training/meshes/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 scale=1 1 1
- added link back_right_foot, mass 0.01; collision mesh filename=/home/matthewthomasbeck/Projects/Robot_Dog/training/meshes/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 scale=1 1 1; visual mesh filename=/home/matthewthomasbeck/Projects/Robot_Dog/training/meshes/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 scale=1 1 1
- added link back_right_hip, mass 0.01; collision mesh filename=/home/matthewthomasbeck/Projects/Robot_Dog/training/meshes/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 scale=1 1 1; visual mesh filename=/home/matthewthomasbeck/Projects/Robot_Dog/training/meshes/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 scale=1 1 1
- added link back_right_pelvis_disc, mass 0.01; collision mesh filename=/home/matthewthomasbeck/Projects/Robot_Dog/training/meshes/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 scale=1 1 1; visual mesh filename=/home/matthewthomasbeck/Projects/Robot_Dog/training/meshes/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 scale=1 1 1
- added link back_right_pelvis_pelvis, mass 0.01; collision mesh filename=/home/matthewthomasbeck/Projects/Robot_Dog/training/meshes/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 scale=1 1 1; visual mesh filename=/home/matthewthomasbeck/Projects/Robot_Dog/training/meshes/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 scale=1 1 1
- added link back_right_pelvis_servo, mass 0.01; collision mesh filename=/home/matthewthomasbeck/Projects/Robot_Dog/training/meshes/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 scale=1 1 1; visual mesh filename=/home/matthewthomasbeck/Projects/Robot_Dog/training/meshes/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 scale=1 1 1
- added link back_right_shin_horn, mass 0.01; collision mesh filename=/home/matthewthomasbeck/Projects/Robot_Dog/training/meshes/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 scale=1 1 1; visual mesh filename=/home/matthewthomasbeck/Projects/Robot_Dog/training/meshes/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 scale=1 1 1
- added link back_right_shin_servo, mass 0.01; collision mesh filename=/home/matthewthomasbeck/Projects/Robot_Dog/training/meshes/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 scale=1 1 1; visual mesh filename=/home/matthewthomasbeck/Projects/Robot_Dog/training/meshes/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 scale=1 1 1
- added link back_right_shin_shin, mass 0.01; collision mesh filename=/home/matthewthomasbeck/Projects/Robot_Dog/training/meshes/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 scale=1 1 1; visual mesh filename=/home/matthewthomasbeck/Projects/Robot_Dog/training/meshes/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 scale=1 1 1
- added link back_top, mass 0.01; collision mesh filename=/home/matthewthomasbeck/Projects/Robot_Dog/training/meshes/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 scale=1 1 1; visual mesh filename=/home/matthewthomasbeck/Projects/Robot_Dog/training/meshes/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 scale=1 1 1
- added link front_face, mass 0.01; collision mesh filename=/home/matthewthomasbeck/Projects/Robot_Dog/training/meshes/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 scale=1 1 1; visual mesh filename=/home/matthewthomasbeck/Projects/Robot_Dog/training/meshes/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 scale=1 1 1
- added link front_left_femur_disc, mass 0.01; collision mesh filename=/home/matthewthomasbeck/Projects/Robot_Dog/training/meshes/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 scale=1 1 1; visual mesh filename=/home/matthewthomasbeck/Projects/Robot_Dog/training/meshes/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 scale=1 1 1
- added link front_left_femur_femur, mass 0.01; collision mesh filename=/home/matthewthomasbeck/Projects/Robot_Dog/training/meshes/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 scale=1 1 1; visual mesh filename=/home/matthewthomasbeck/Projects/Robot_Dog/training/meshes/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 scale=1 1 1
- added link front_left_femur_servo, mass 0.01; collision mesh filename=/home/matthewthomasbeck/Projects/Robot_Dog/training/meshes/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 scale=1 1 1; visual mesh filename=/home/matthewthomasbeck/Projects/Robot_Dog/training/meshes/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 scale=1 1 1
- added link front_left_foot, mass 0.01; collision mesh filename=/home/matthewthomasbeck/Projects/Robot_Dog/training/meshes/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 scale=1 1 1; visual mesh filename=/home/matthewthomasbeck/Projects/Robot_Dog/training/meshes/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 scale=1 1 1
- added link front_left_hip, mass 0.01; collision mesh filename=/home/matthewthomasbeck/Projects/Robot_Dog/training/meshes/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 scale=1 1 1; visual mesh filename=/home/matthewthomasbeck/Projects/Robot_Dog/training/meshes/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 scale=1 1 1
- added link front_left_pelvis_disc, mass 0.01; collision mesh filename=/home/matthewthomasbeck/Projects/Robot_Dog/training/meshes/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 scale=1 1 1; visual mesh filename=/home/matthewthomasbeck/Projects/Robot_Dog/training/meshes/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 scale=1 1 1
- added link front_left_pelvis_pelvis, mass 0.01; collision mesh filename=/home/matthewthomasbeck/Projects/Robot_Dog/training/meshes/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 scale=1 1 1; visual mesh filename=/home/matthewthomasbeck/Projects/Robot_Dog/training/meshes/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 scale=1 1 1
- added link front_left_pelvis_servo, mass 0.01; collision mesh filename=/home/matthewthomasbeck/Projects/Robot_Dog/training/meshes/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 scale=1 1 1; visual mesh filename=/home/matthewthomasbeck/Projects/Robot_Dog/training/meshes/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 scale=1 1 1
- added link front_left_shin_horn, mass 0.01; collision mesh filename=/home/matthewthomasbeck/Projects/Robot_Dog/training/meshes/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 scale=1 1 1; visual mesh filename=/home/matthewthomasbeck/Projects/Robot_Dog/training/meshes/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 scale=1 1 1
- added link front_left_shin_servo, mass 0.01; collision mesh filename=/home/matthewthomasbeck/Projects/Robot_Dog/training/meshes/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 scale=1 1 1; visual mesh filename=/home/matthewthomasbeck/Projects/Robot_Dog/training/meshes/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 scale=1 1 1
- added link front_left_shin_shin, mass 0.01; collision mesh filename=/home/matthewthomasbeck/Projects/Robot_Dog/training/meshes/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 scale=1 1 1; visual mesh filename=/home/matthewthomasbeck/Projects/Robot_Dog/training/meshes/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 scale=1 1 1
- added link front_right_femur_disc, mass 0.01; collision mesh filename=/home/matthewthomasbeck/Projects/Robot_Dog/training/meshes/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 scale=1 1 1; visual mesh filename=/home/matthewthomasbeck/Projects/Robot_Dog/training/meshes/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 scale=1 1 1
- added link front_right_femur_femur, mass 0.01; collision mesh filename=/home/matthewthomasbeck/Projects/Robot_Dog/training/meshes/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 scale=1 1 1; visual mesh filename=/home/matthewthomasbeck/Projects/Robot_Dog/training/meshes/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 scale=1 1 1
- added link front_right_femur_servo, mass 0.01; collision mesh filename=/home/matthewthomasbeck/Projects/Robot_Dog/training/meshes/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 scale=1 1 1; visual mesh filename=/home/matthewthomasbeck/Projects/Robot_Dog/training/meshes/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 scale=1 1 1
- added link front_right_foot, mass 0.01; collision mesh filename=/home/matthewthomasbeck/Projects/Robot_Dog/training/meshes/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 scale=1 1 1; visual mesh filename=/home/matthewthomasbeck/Projects/Robot_Dog/training/meshes/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 scale=1 1 1
- added link front_right_hip, mass 0.01; collision mesh filename=/home/matthewthomasbeck/Projects/Robot_Dog/training/meshes/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 scale=1 1 1; visual mesh filename=/home/matthewthomasbeck/Projects/Robot_Dog/training/meshes/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 scale=1 1 1
- added link front_right_pelvis_disc, mass 0.01; collision mesh filename=/home/matthewthomasbeck/Projects/Robot_Dog/training/meshes/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 scale=1 1 1; visual mesh filename=/home/matthewthomasbeck/Projects/Robot_Dog/training/meshes/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 scale=1 1 1
- added link front_right_pelvis_pelvis, mass 0.01; collision mesh filename=/home/matthewthomasbeck/Projects/Robot_Dog/training/meshes/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 scale=1 1 1; visual mesh filename=/home/matthewthomasbeck/Projects/Robot_Dog/training/meshes/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 scale=1 1 1
- added link front_right_pelvis_servo, mass 0.01; collision mesh filename=/home/matthewthomasbeck/Projects/Robot_Dog/training/meshes/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 scale=1 1 1; visual mesh filename=/home/matthewthomasbeck/Projects/Robot_Dog/training/meshes/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 scale=1 1 1
- added link front_right_shin_horn, mass 0.01; collision mesh filename=/home/matthewthomasbeck/Projects/Robot_Dog/training/meshes/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 scale=1 1 1; visual mesh filename=/home/matthewthomasbeck/Projects/Robot_Dog/training/meshes/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 scale=1 1 1
- added link front_right_shin_servo, mass 0.01; collision mesh filename=/home/matthewthomasbeck/Projects/Robot_Dog/training/meshes/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 scale=1 1 1; visual mesh filename=/home/matthewthomasbeck/Projects/Robot_Dog/training/meshes/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 scale=1 1 1
- added link front_right_shin_shin, mass 0.01; collision mesh filename=/home/matthewthomasbeck/Projects/Robot_Dog/training/meshes/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 scale=1 1 1; visual mesh filename=/home/matthewthomasbeck/Projects/Robot_Dog/training/meshes/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 scale=1 1 1
- added link front_top, mass 0.01; collision mesh filename=/home/matthewthomasbeck/Projects/Robot_Dog/training/meshes/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 scale=1 1 1; visual mesh filename=/home/matthewthomasbeck/Projects/Robot_Dog/training/meshes/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 scale=1 1 1
- added link midsection_batteryplate, mass 0.01; collision mesh filename=/home/matthewthomasbeck/Projects/Robot_Dog/training/meshes/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 scale=1 1 1; visual mesh filename=/home/matthewthomasbeck/Projects/Robot_Dog/training/meshes/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 scale=1 1 1
- added link midsection_bottom, mass 0.01; collision mesh filename=/home/matthewthomasbeck/Projects/Robot_Dog/training/meshes/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 scale=1 1 1; visual mesh filename=/home/matthewthomasbeck/Projects/Robot_Dog/training/meshes/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 scale=1 1 1
- added link midsection_connectorplate, mass 0.01; collision mesh filename=/home/matthewthomasbeck/Projects/Robot_Dog/training/meshes/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 scale=1 1 1; visual mesh filename=/home/matthewthomasbeck/Projects/Robot_Dog/training/meshes/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 scale=1 1 1
- added link midsection_side_left, mass 0.01; collision mesh filename=/home/matthewthomasbeck/Projects/Robot_Dog/training/meshes/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 scale=1 1 1; visual mesh filename=/home/matthewthomasbeck/Projects/Robot_Dog/training/meshes/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 scale=1 1 1
- added link midsection_side_right, mass 0.01; collision mesh filename=/home/matthewthomasbeck/Projects/Robot_Dog/training/meshes/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 scale=1 1 1; visual mesh filename=/home/matthewthomasbeck/Projects/Robot_Dog/training/meshes/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 scale=1 1 1
- added link midsection_top, mass 0.01; collision mesh filename=/home/matthewthomasbeck/Projects/Robot_Dog/training/meshes/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 scale=1 1 1; visual mesh filename=/home/matthewthomasbeck/Projects/Robot_Dog/training/meshes/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 scale=1 1 1
- link battery: geometry collision mesh filename=/home/matthewthomasbeck/Projects/Robot_Dog/training/meshes/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 scale=1 1 1; visual mesh filename=/home/matthewthomasbeck/Projects/Robot_Dog/training/meshes/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 scale=1 1 1
Joints:
- removed joint ai_module/midsection-connectorplate
- removed joint back-butt/back-top
- removed joint back-left-femur-disc/femur
- removed joint back-left-femur-servo/back-left-hip
- removed joint back-left-pelvis-disc/pelvis
- removed joint back-left-pelvis-pelvis/back-left-femur-servo
- removed joint back-left-pelvis-pelvis/back-left-shin-servo
- removed joint back-left-shin-servo/horn
- removed joint back-left-shin-shin/back-left-foot
- removed joint back-right-femur-disc/femur
- removed joint back-right-femur-servo/back-right-hip
- removed joint back-right-pelvis-disc/pelvis
- removed joint back-right-pelvis-pelvis/back-right-femur-servo
- removed joint back-right-pelvis-pelvis/back-right-shin-servo
- removed joint back-right-shin-servo/horn
- removed joint back-right-shin-shin/back-right-foot
- removed joint battery/midsection-batteryplate
- removed joint front-face/top
- removed joint front-left-femur-disc/femur
- removed joint front-left-femur-servo/front-left-hip
- removed joint front-left-pelvis-disc/pelvis
- removed joint front-left-pelvis-pelvis/front-left-femur-servo
- removed joint front-left-pelvis-pelvis/front-left-shin-servo
- removed joint front-left-shin-servo/horn
- removed joint front-left-shin-shin/front-left-foot
- removed joint front-right-femur-disc/femur
- removed joint front-right-femur-servo/front-right-hip
- removed joint front-right-pelvis-disc/pelvis
- removed joint front-right-pelvis-pelvis/front-right-femur-servo
- removed joint front-right-pelvis-pelvis/front-right-shin-servo
- removed joint front-right-shin-servo/horn
- removed joint front-right-shin-shin/front-right-foot
- removed joint midsection-bottom/back-butt
- removed joint midsection-bottom/back-left-pelvis-servo
- removed joint midsection-bottom/back-right-pelvis-servo
- removed joint midsection-bottom/connectorplate
- removed joint midsection-bottom/front-face
- removed joint midsection-bottom/front-left-pelvis-servo
- removed joint midsection-bottom/front-right-pelvis-servo
- removed joint midsection-bottom/side-left
- removed joint midsection-bottom/side-right
- removed joint midsection-bottom/top
- removed joint midsection-top/batteryplate
- added joint ai_module_midsection_connectorplate: type fixed, parent midsection_connectorplate, child ai_module_mock, origin xyz=-0.00726 -0.074 0.0162 rpy=0 0 3.14
- added joint back_butt_back_top: type fixed, parent back_butt, child back_top, origin xyz=-0.0097 -1.118 -0.6045 rpy=0 0 3.14
- added joint back_left_femur_disc_femur: type fixed, parent back_left_femur_disc, child back_left_femur_femur, origin xyz=0 0 0 rpy=0 -1.5708 3.14
- added joint back_left_femur_servo_back_left_hip: type continuous, parent back_left_femur_servo, child back_left_hip, origin xyz=0 -0.01 0.0409 rpy=0 -1.5708 3.14
- added joint back_left_pelvis_disc_pelvis: type fixed, parent back_left_pelvis_disc, child back_left_pelvis_pelvis, origin xyz=0 0.0425 0.00413 rpy=-1.5708 0 0
- added joint back_left_pelvis_pelvis_back_left_femur_servo: type fixed, parent back_left_pelvis_pelvis, child back_left_femur_servo, origin xyz=-0.0175 -0.0271 -0.0431 rpy=1.5708 1.5708 1.5708
- added joint back_left_pelvis_pelvis_back_left_shin_servo: type fixed, parent back_left_pelvis_pelvis, child back_left_shin_servo, origin xyz=-0.0175 -0.0271 -0.0231 rpy=1.5708 -1.5708 1.5708
- added joint back_left_shin_servo_horn: type continuous, parent back_left_shin_servo, child back_left_shin_horn, origin xyz=0 -0.01 0.043 rpy=0 0 0.785398, axis 0 0 1
- added joint back_left_shin_shin_back_left_foot: type fixed, parent back_left_shin_shin, child back_left_foot, origin xyz=-0.0367 -0.06 0.035 rpy=0 0 0
- added joint back_right_femur_disc_femur: type fixed, parent back_right_femur_disc, child back_right_femur_femur, origin xyz=0 0 0 rpy=0 1.5708 3.14
- added joint back_right_femur_servo_back_right_hip: type continuous, parent back_right_femur_servo, child back_right_hip, origin xyz=0 -0.01 0.0468 rpy=0 1.5708 3.14
- added joint back_right_pelvis_disc_pelvis: type fixed, parent back_right_pelvis_disc, child back_right_pelvis_pelvis, origin xyz=0 0.0425 0.00413 rpy=-1.5708 0 3.14
- added joint back_right_pelvis_pelvis_back_right_femur_servo: type fixed, parent back_right_pelvis_pelvis, child back_right_femur_servo, origin xyz=-0.0175 -0.0271 0.0431 rpy=1.5708 1.5708 1.5708
- added joint back_right_pelvis_pelvis_back_right_shin_servo: type fixed, parent back_right_pelvis_pelvis, child back_right_shin_servo, origin xyz=-0.0175 -0.0271 0.0231 rpy=1.5708 -1.5708 1.5708
- added joint back_right_shin_servo_horn: type continuous, parent back_right_shin_servo, child back_right_shin_horn, origin xyz=0 -0.01 0.043 rpy=0 0 2.356198, axis 0 0 1
- added joint back_right_shin_shin_back_right_foot: type fixed, parent back_right_shin_shin, child back_right_foot, origin xyz=-0.04258 -0.06 0.035 rpy=0 0 0
- added joint battery_midsection_batteryplate: type fixed, parent midsection_batteryplate, child battery, origin xyz=0.007 0.077 -0.0012 rpy=1.5708 0 0
- added joint front_face_top: type fixed, parent front_face, child front_top, origin xyz=0.514 -0.042 0.07945 rpy=0 0 3.14
- added joint front_left_femur_disc_femur: type fixed, parent front_left_femur_disc, child front_left_femur_femur, origin xyz=0 0 0 rpy=0 -1.5708 3.14
- added joint front_left_femur_servo_front_left_hip: type continuous, parent front_left_femur_servo, child front_left_hip, origin xyz=0 -0.01 0.0409 rpy=0 -1.5708 3.14
- added joint front_left_pelvis_disc_pelvis: type fixed, parent front_left_pelvis_disc, child front_left_pelvis_pelvis, origin xyz=0 0.0425 0.00413 rpy=-1.5708 0 3.14
- added joint front_left_pelvis_pelvis_front_left_femur_servo: type fixed, parent front_left_pelvis_pelvis, child front_left_femur_servo, origin xyz=-0.0175 -0.0271 0.0431 rpy=0 -1.5708 -3.14
- added joint front_left_pelvis_pelvis_front_left_shin_servo: type fixed, parent front_left_pelvis_pelvis, child front_left_shin_servo, origin xyz=-0.0175 -0.0271 0.0231 rpy=-1.5708 1.5708 -1.5708
- added joint front_left_shin_servo_horn: type continuous, parent front_left_shin_servo, child front_left_shin_horn, origin xyz=0 -0.01 0.043 rpy=0 0 0.785398, axis 0 0 1
- added joint front_left_shin_shin_front_left_foot: type fixed, parent front_left_shin_shin, child front_left_foot, origin xyz=-0.0367 -0.06 0.035 rpy=0 0 0
- added joint front_right_femur_disc_femur: type fixed, parent front_right_femur_disc, child front_right_femur_femur, origin xyz=0 0 0 rpy=0 1.5708 3.14
- added joint front_right_femur_servo_front_right_hip: type continuous, parent front_right_femur_servo, child front_right_hip, origin xyz=0 -0.01 0.0468 rpy=0 1.5708 3.14
- added joint front_right_pelvis_disc_pelvis: type fixed, parent front_right_pelvis_disc, child front_right_pelvis_pelvis, origin xyz=0 0.0425 0.00413 rpy=-1.5708 0 0
- added joint front_right_pelvis_pelvis_front_right_femur_servo: type fixed, parent front_right_pelvis_pelvis, child front_right_femur_servo, origin xyz=-0.0175 -0.0271 -0.0431 rpy=0 -1.5708 -3.14
- added joint front_right_pelvis_pelvis_front_right_shin_servo: type fixed, parent front_right_pelvis_pelvis, child front_right_shin_servo, origin xyz=-0.0175 -0.0271 -0.0231 rpy=1.5708 1.5708 1.5708
- added joint front_right_shin_servo_horn: type continuous, parent front_right_shin_servo, child front_right_shin_horn, origin xyz=0 -0.01 0.043 rpy=0 0 2.356198, axis 0 0 1
- added joint front_right_shin_shin_front_right_foot: type fixed, parent front_right_shin_shin, child front_right_foot, origin xyz=-0.04258 -0.06 0.035 rpy=0 0 0
- added joint midsection_bottom_back_butt: type fixed, parent midsection_bottom, child back_butt, origin xyz=-0.117 -0.394 -0.026 rpy=0 0 3.14
- added joint midsection_bottom_back_left_pelvis_servo: type fixed, parent midsection_bottom, child back_left_pelvis_servo, origin xyz=0.0005 0.0785 0.0333 rpy=1.5708 3.14 3.14
- added joint midsection_bottom_back_right_pelvis_servo: type fixed, parent midsection_bottom, child back_right_pelvis_servo, origin xyz=-0.0975 0.0785 0.0333 rpy=1.5708 3.14 3.14
- added joint midsection_bottom_connectorplate: type fixed, parent midsection_bottom, child midsection_connectorplate, origin xyz=0.002 0.2 0.008 rpy=0 0 0
- added joint midsection_bottom_front_face: type fixed, parent midsection_bottom, child front_face, origin xyz=0.514 -0.043 -0.0794 rpy=0 0 3.14
- added joint midsection_bottom_front_left_pelvis_servo: type fixed, parent midsection_bottom, child front_left_pelvis_servo, origin xyz=0.0005 0.05 0.0333 rpy=1.5708 3.14 0
- added joint midsection_bottom_front_right_pelvis_servo: type fixed, parent midsection_bottom, child front_right_pelvis_servo, origin xyz=-0.0975 0.05 0.0333 rpy=1.5708 3.14 0
- added joint midsection_bottom_side_left: type fixed, parent midsection_bottom, child midsection_side_left, origin xyz=0 0 0 rpy=0 0 0
- added joint midsection_bottom_side_right: type fixed, parent midsection_bottom, child midsection_side_right, origin xyz=-0.09705 0.1283 0 rpy=0 0 3.14
- added joint midsection_bottom_top: type fixed, parent midsection_bottom, child midsection_top, origin xyz=0 0 0 rpy=0 0 0
- added joint midsection_top_batteryplate: type fixed, parent midsection_top, child midsection_batteryplate, origin xyz=-0.056 0.057 0.09855 rpy=0 0 0
- joint BL_hip: child back-left-pelvis-disc -> back_left_pelvis_disc; parent back-left-pelvis-servo -> back_left_pelvis_servo
- joint BL_lower: child back-left-shin-shin -> back_left_shin_shin; parent back-left-femur-femur -> back_left_femur_femur
- joint BL_upper: child back-left-femur-disc -> back_left_femur_disc; parent back-left-femur-servo -> back_left_femur_servo
- joint BR_hip: child back-right-pelvis-disc -> back_right_pelvis_disc; parent back-right-pelvis-servo -> back_right_pelvis_servo
- joint BR_lower: child back-right-shin-shin -> back_right_shin_shin; parent back-right-femur-femur -> back_right_femur_femur
- joint BR_upper: child back-right-femur-disc -> back_right_femur_disc; parent back-right-femur-servo -> back_right_femur_servo
- joint FL_hip: child front-left-pelvis-disc -> front_left_pelvis_disc; parent front-left-pelvis-servo -> front_left_pelvis_servo
- joint FL_lower: child front-left-shin-shin -> front_left_shin_shin; parent front-left-femur-femur -> front_left_femur_femur
- joint FL_upper: child front-left-femur-disc -> front_left_femur_disc; parent front-left-femur-servo -> front_left_femur_servo
- joint FR_hip: child front-right-pelvis-disc -> front_right_pelvis_disc; parent front-right-pelvis-servo -> front_right_pelvis_servo
- joint FR_lower: child front-right-shin-shin -> front_right_shin_shin; parent front-right-femur-femur -> front_right_femur_femur
- joint FR_upper: child front-right-femur-disc -> front_right_femur_disc; parent front-right-femur-servo -> front_right_femur_servo
