Commit message: Changed the urdf to have no joint restriction

File: training/urdf/robot_dog.urdf (robot description, URDF)
Before this commit: robot Robot_Dog, 48 links, 47 joints
Joints:
- joint BL_hip: limit lower=-0.349066 upper=0.349066 effort=5.0 velocity=9.52 -> lower=-3.14159 upper=3.14159 effort=5.0 velocity=9.52
- joint BL_lower: limit lower=-0.698 upper=0.698 effort=5.0 velocity=9.52 -> lower=-3.14159 upper=3.14159 effort=5.0 velocity=9.52
- joint BL_upper: limit lower=-0.654 upper=0.654 effort=5.0 velocity=9.52 -> lower=-3.14159 upper=3.14159 effort=5.0 velocity=9.52
- joint BR_hip: limit lower=-0.349066 upper=0.349066 effort=5.0 velocity=9.52 -> lower=-3.14159 upper=3.14159 effort=5.0 velocity=9.52
- joint BR_lower: limit lower=-0.698 upper=0.698 effort=5.0 velocity=9.52 -> lower=-3.14159 upper=3.14159 effort=5.0 velocity=9.52
- joint BR_upper: limit lower=-0.654 upper=0.654 effort=5.0 velocity=9.52 -> lower=-3.14159 upper=3.14159 effort=5.0 velocity=9.52
- joint FL_hip: limit lower=-0.349066 upper=0.349066 effort=5.0 velocity=9.52 -> lower=-3.14159 upper=3.14159 effort=5.0 velocity=9.52
- joint FL_lower: limit lower=-0.698 upper=0.698 effort=5.0 velocity=9.52 -> lower=-3.14159 upper=3.14159 effort=5.0 velocity=9.52
- joint FL_upper: limit lower=-0.654 upper=0.654 effort=5.0 velocity=9.52 -> lower=-3.14159 upper=3.14159 effort=5.0 velocity=9.52
- joint FR_hip: limit lower=-0.349066 upper=0.349066 effort=5.0 velocity=9.52 -> lower=-3.14159 upper=3.14159 effort=5.0 velocity=9.52
- joint FR_lower: limit lower=-0.698 upper=0.698 effort=5.0 velocity=9.52 -> lower=-3.14159 upper=3.14159 effort=5.0 velocity=9.52
- joint FR_upper: limit lower=-0.654 upper=0.654 effort=5.0 velocity=9.52 -> lower=-3.14159 upper=3.14159 effort=5.0 velocity=9.52

Commit message: Calibration completely accurate

File: training/urdf/robot_dog.urdf (robot description, URDF)
Before this commit: robot Robot_Dog, 48 links, 47 joints
Joints:
- joint BL_hip: axis 0 0 1 -> 0 0 -1
- joint BL_lower: axis 1 0 0 -> -1 0 0
- joint BL_upper: axis 0 0 1 -> 0 0 -1
- joint FL_lower: axis 1 0 0 -> -1 0 0
- joint FR_hip: axis 0 0 1 -> 0 0 -1

Commit message: Isaac Sim successfully mapped!

File: training/urdf/robot_dog.urdf (robot description, URDF)
Before this commit: robot Robot_Dog, 48 links, 47 joints
Joints:
- joint BL_hip: axis 0 0 -1 -> 0 0 1
- joint BL_lower: axis -1 0 0 -> 1 0 0
- joint BL_upper: axis 0 0 -1 -> 0 0 1
- joint FL_lower: axis -1 0 0 -> 1 0 0
- joint FR_hip: axis 0 0 -1 -> 0 0 1

Commit message: Finally got a training loop going, added masses to urdf

File: training/urdf/robot_dog.urdf (robot description, URDF)
Before this commit: robot Robot_Dog, 48 links, 47 joints
Links:
- link ai_module_mock: mass 0.01 -> 0.4
- link back_butt: mass 0.01 -> 0.035
- link back_left_femur_disc: mass 0.01 -> 0.002
- link back_left_femur_femur: mass 0.01 -> 0.015
- link back_left_femur_servo: mass 0.01 -> 0.07
- link back_left_foot: mass 0.01 -> 0.008
- link back_left_pelvis_disc: mass 0.01 -> 0.002
- link back_left_pelvis_pelvis: mass 0.01 -> 0.004
- link back_left_pelvis_servo: mass 0.01 -> 0.07
- link back_left_shin_servo: mass 0.01 -> 0.07
- link back_left_shin_shin: mass 0.01 -> 0.009
- link back_right_femur_disc: mass 0.01 -> 0.002
- link back_right_femur_femur: mass 0.01 -> 0.015
- link back_right_femur_servo: mass 0.01 -> 0.07
- link back_right_foot: mass 0.01 -> 0.008
- link back_right_pelvis_disc: mass 0.01 -> 0.002
- link back_right_pelvis_pelvis: mass 0.01 -> 0.004
- link back_right_pelvis_servo: mass 0.01 -> 0.07
- link back_right_shin_servo: mass 0.01 -> 0.07
- link back_right_shin_shin: mass 0.01 -> 0.009
- link back_top: mass 0.01 -> 0.017
- link battery: mass 0.01 -> 0.3
- link front_face: mass 0.01 -> 0.035
- link front_left_femur_disc: mass 0.01 -> 0.002
- link front_left_femur_femur: mass 0.01 -> 0.015
- link front_left_femur_servo: mass 0.01 -> 0.07
- link front_left_foot: mass 0.01 -> 0.008
- link front_left_pelvis_disc: mass 0.01 -> 0.002
- link front_left_pelvis_pelvis: mass 0.01 -> 0.004
- link front_left_pelvis_servo: mass 0.01 -> 0.07
- link front_left_shin_servo: mass 0.01 -> 0.07
- link front_left_shin_shin: mass 0.01 -> 0.009
- link front_right_femur_disc: mass 0.01 -> 0.002
- link front_right_femur_femur: mass 0.01 -> 0.015
- link front_right_femur_servo: mass 0.01 -> 0.07
- link front_right_foot: mass 0.01 -> 0.008
- link front_right_pelvis_disc: mass 0.01 -> 0.002
- link front_right_pelvis_pelvis: mass 0.01 -> 0.004
- link front_right_pelvis_servo: mass 0.01 -> 0.07
- link front_right_shin_servo: mass 0.01 -> 0.07
- link front_right_shin_shin: mass 0.01 -> 0.009
- link front_top: mass 0.01 -> 0.017
- link midsection_batteryplate: mass 0.01 -> 0.022
- link midsection_bottom: mass 0.01 -> 0.089
- link midsection_connectorplate: mass 0.01 -> 0.020
- link midsection_side_left: mass 0.01 -> 0.023
- link midsection_side_right: mass 0.01 -> 0.023
- link midsection_top: mass 0.01 -> 0.042

Commit message: Saving checkpoint, going to see why velocity is giving me such massive problems in issac

File: training/urdf/robot_dog.urdf (robot description, URDF)
Before this commit: robot Robot_Dog, 48 links, 47 joints
Links:
- link back_left_pelvis_pelvis: mass 0.004 -> 0.017
- link back_right_pelvis_pelvis: mass 0.004 -> 0.017
- link front_left_pelvis_pelvis: mass 0.004 -> 0.017
- link front_right_pelvis_pelvis: mass 0.004 -> 0.017
Joints:
- joint BL_lower: limit lower=-3.14159 upper=3.14159 effort=5.0 velocity=9.52 -> lower=-3.14159 upper=3.14159 effort=5.0 velocity=3.173
- joint BR_lower: limit lower=-3.14159 upper=3.14159 effort=5.0 velocity=9.52 -> lower=-3.14159 upper=3.14159 effort=5.0 velocity=3.173
- joint FL_lower: limit lower=-3.14159 upper=3.14159 effort=5.0 velocity=9.52 -> lower=-3.14159 upper=3.14159 effort=5.0 velocity=3.173
- joint FR_lower: limit lower=-3.14159 upper=3.14159 effort=5.0 velocity=9.52 -> lower=-3.14159 upper=3.14159 effort=5.0 velocity=3.173

Commit message: Made the joint torques realistic

File: training/urdf/robot_dog.urdf (robot description, URDF)
Before this commit: robot Robot_Dog, 48 links, 47 joints
Joints:
- joint BL_hip: limit lower=-3.14159 upper=3.14159 effort=5.0 velocity=9.52 -> lower=-3.14159 upper=3.14159 effort=4.4 velocity=9.52
- joint BL_lower: limit lower=-3.14159 upper=3.14159 effort=5.0 velocity=3.173 -> lower=-3.14159 upper=3.14159 effort=4.4 velocity=9.52
- joint BL_upper: limit lower=-3.14159 upper=3.14159 effort=5.0 velocity=9.52 -> lower=-3.14159 upper=3.14159 effort=4.4 velocity=9.52
- joint BR_hip: limit lower=-3.14159 upper=3.14159 effort=5.0 velocity=9.52 -> lower=-3.14159 upper=3.14159 effort=4.4 velocity=9.52
- joint BR_lower: limit lower=-3.14159 upper=3.14159 effort=5.0 velocity=3.173 -> lower=-3.14159 upper=3.14159 effort=4.4 velocity=9.52
- joint BR_upper: limit lower=-3.14159 upper=3.14159 effort=5.0 velocity=9.52 -> lower=-3.14159 upper=3.14159 effort=4.4 velocity=9.52
- joint FL_hip: limit lower=-3.14159 upper=3.14159 effort=5.0 velocity=9.52 -> lower=-3.14159 upper=3.14159 effort=4.4 velocity=9.52
- joint FL_lower: limit lower=-3.14159 upper=3.14159 effort=5.0 velocity=3.173 -> lower=-3.14159 upper=3.14159 effort=4.4 velocity=9.52
- joint FL_upper: limit lower=-3.14159 upper=3.14159 effort=5.0 velocity=9.52 -> lower=-3.14159 upper=3.14159 effort=4.4 velocity=9.52
- joint FR_hip: limit lower=-3.14159 upper=3.14159 effort=5.0 velocity=9.52 -> lower=-3.14159 upper=3.14159 effort=4.4 velocity=9.52
- joint FR_lower: limit lower=-3.14159 upper=3.14159 effort=5.0 velocity=3.173 -> lower=-3.14159 upper=3.14159 effort=4.4 velocity=9.52
- joint FR_upper: limit lower=-3.14159 upper=3.14159 effort=5.0 velocity=9.52 -> lower=-3.14159 upper=3.14159 effort=4.4 velocity=9.52

Commit message: Made distal movement half as fast as proximal for realistic actuation (because the servos that control the lower parts of the legs are top-mounted, they dont get twice the leverage an animals leg normally would... *sicence*)

File: training/urdf/robot_dog.urdf (robot description, URDF)
Before this commit: robot Robot_Dog, 48 links, 47 joints
Joints:
- joint BL_lower: limit lower=-3.14159 upper=3.14159 effort=4.4 velocity=9.52 -> lower=-3.14159 upper=3.14159 effort=4.4 velocity=4.76
- joint BR_lower: limit lower=-3.14159 upper=3.14159 effort=4.4 velocity=9.52 -> lower=-3.14159 upper=3.14159 effort=4.4 velocity=4.76
- joint FL_lower: limit lower=-3.14159 upper=3.14159 effort=4.4 velocity=9.52 -> lower=-3.14159 upper=3.14159 effort=4.4 velocity=4.76
- joint FR_lower: limit lower=-3.14159 upper=3.14159 effort=4.4 velocity=9.52 -> lower=-3.14159 upper=3.14159 effort=4.4 velocity=4.76
